File: mk1/mk1.kicad_pcb (KiCad board)
At the start: 2 copper layers, 230 x 70 mm, 1 part, among them U1 STM32F070CBTx

Commit message: using ML switch built i jumper bar
Parts:
- added D1: 1N4148, Diode_SMD:D_SOD-123, B.Cu at (55.0, 61.0)
- added D10: 1N4148, Diode_SMD:D_SOD-123, B.Cu at (51.0, 113.0)
- added D11: 1N4148, Diode_SMD:D_SOD-123, B.Cu at (88.0, 56.0)
- added D12: 1N4148, Diode_SMD:D_SOD-123, B.Cu at (83.0, 69.0)
- added D13: 1N4148, Diode_SMD:D_SOD-123, B.Cu at (78.0, 82.0)
- added D14: 1N4148, Diode_SMD:D_SOD-123, B.Cu at (73.0, 95.0)
- added D15: 1N4148, Diode_SMD:D_SOD-123, B.Cu at (68.0, 108.0)
- added D16: 1N4148, Diode_SMD:D_SOD-123, B.Cu at (104.0, 56.0)
- added D17: 1N4148, Diode_SMD:D_SOD-123, B.Cu at (99.0, 69.0)
- added D18: 1N4148, Diode_SMD:D_SOD-123, B.Cu at (94.0, 82.0)
- added D19: 1N4148, Diode_SMD:D_SOD-123, B.Cu at (89.0, 95.0)
- added D2: 1N4148, Diode_SMD:D_SOD-123, B.Cu at (50.4, 74.0)
- added D20: 1N4148, Diode_SMD:D_SOD-123, B.Cu at (84.0, 108.0)
- added D21: 1N4148, Diode_SMD:D_SOD-123, B.Cu at (117.0, 63.0)
- added D22: 1N4148, Diode_SMD:D_SOD-123, B.Cu at (112.0, 76.0)
- added D23: 1N4148, Diode_SMD:D_SOD-123, B.Cu at (107.0, 89.0)
- added D24: 1N4148, Diode_SMD:D_SOD-123, B.Cu at (102.0, 102.0)
- added D25: 1N4148, Diode_SMD:D_SOD-123, B.Cu at (97.0, 115.0)
- added D26: 1N4148, Diode_SMD:D_SOD-123, B.Cu at (131.7, 68.0)
- added D27: 1N4148, Diode_SMD:D_SOD-123, B.Cu at (126.0, 81.0)
- added D28: 1N4148, Diode_SMD:D_SOD-123, B.Cu at (121.0, 94.0)
- added D29: 1N4148, Diode_SMD:D_SOD-123, B.Cu at (116.0, 107.0)
- added D3: 1N4148, Diode_SMD:D_SOD-123, B.Cu at (45.0, 87.0)
- added D30: 1N4148, Diode_SMD:D_SOD-123, B.Cu at (111.0, 120.0)
- added D31: 1N4148, Diode_SMD:D_SOD-123, B.Cu at (165.0, 71.0)
- added D32: 1N4148, Diode_SMD:D_SOD-123, B.Cu at (166.0, 89.0)
- added D33: 1N4148, Diode_SMD:D_SOD-123, B.Cu at (173.0, 104.0)
- added D34: 1N4148, Diode_SMD:D_SOD-123, B.Cu at (174.0, 116.0)
- added D35: 1N4148, Diode_SMD:D_SOD-123, B.Cu at (180.0, 131.0)
- added D36: 1N4148, Diode_SMD:D_SOD-123, B.Cu at (178.0, 71.0)
- added D37: 1N4148, Diode_SMD:D_SOD-123, B.Cu at (189.0, 89.0)
- added D38: 1N4148, Diode_SMD:D_SOD-123, B.Cu at (195.0, 102.0)
- added D39: 1N4148, Diode_SMD:D_SOD-123, B.Cu at (195.0, 117.0)
- added D4: 1N4148, Diode_SMD:D_SOD-123, B.Cu at (40.0, 100.0)
- added D40: 1N4148, Diode_SMD:D_SOD-123, B.Cu at (197.0, 135.0)
- added D41: 1N4148, Diode_SMD:D_SOD-123, B.Cu at (202.0, 69.0)
- added D42: 1N4148, Diode_SMD:D_SOD-123, B.Cu at (202.0, 88.0)
- added D43: 1N4148, Diode_SMD:D_SOD-123, B.Cu at (208.0, 103.0)
- added D44: 1N4148, Diode_SMD:D_SOD-123, B.Cu at (216.0, 119.0)
- added D45: 1N4148, Diode_SMD:D_SOD-123, B.Cu at (217.0, 136.0)
- added D46: 1N4148, Diode_SMD:D_SOD-123, B.Cu at (220.0, 68.0)
- added D47: 1N4148, Diode_SMD:D_SOD-123, B.Cu at (222.0, 88.0)
- added D48: 1N4148, Diode_SMD:D_SOD-123, B.Cu at (226.0, 103.0)
- added D49: 1N4148, Diode_SMD:D_SOD-123, B.Cu at (236.0, 119.0)
- added D5: 1N4148, Diode_SMD:D_SOD-123, B.Cu at (35.0, 113.0)
- added D50: 1N4148, Diode_SMD:D_SOD-123, B.Cu at (236.0, 137.0)
- added D51: 1N4148, Diode_SMD:D_SOD-123, B.Cu at (239.0, 68.0)
- added D52: 1N4148, Diode_SMD:D_SOD-123, B.Cu at (239.0, 88.0)
- added D53: 1N4148, Diode_SMD:D_SOD-123, B.Cu at (243.0, 103.0)
- added D54: 1N4148, Diode_SMD:D_SOD-123, B.Cu at (252.0, 121.0)
- added D55: 1N4148, Diode_SMD:D_SOD-123, B.Cu at (253.0, 138.0)
- added D56: 1N4148, Diode_SMD:D_SOD-123, B.Cu at (262.0, 69.0)
- added D57: 1N4148, Diode_SMD:D_SOD-123, B.Cu at (257.0, 88.0)
- added D58: 1N4148, Diode_SMD:D_SOD-123, B.Cu at (262.0, 103.0)
- added D59: 1N4148, Diode_SMD:D_SOD-123, B.Cu at (272.0, 121.0)
- added D6: 1N4148, Diode_SMD:D_SOD-123, B.Cu at (71.0, 61.0)
- added D60: 1N4148, Diode_SMD:D_SOD-123, B.Cu at (274.0, 138.0)
- added D7: 1N4148, Diode_SMD:D_SOD-123, B.Cu at (66.0, 74.0)
- added D8: 1N4148, Diode_SMD:D_SOD-123, B.Cu at (61.0, 87.0)
- added D9: 1N4148, Diode_SMD:D_SOD-123, B.Cu at (56.0, 100.0)
- added U10: CHERRY_ML, Switches:CHERRY_ML, F.Cu at (54.0, 95.0)
- added U11: CHERRY_ML, Switches:CHERRY_ML, F.Cu at (49.0, 108.0)
- added U12: CHERRY_ML, Switches:CHERRY_ML, F.Cu at (86.0, 51.0)
- added U13: CHERRY_ML, Switches:CHERRY_ML, F.Cu at (81.0, 64.0)
- added U14: CHERRY_ML, Switches:CHERRY_ML, F.Cu at (76.0, 77.0)
- added U15: CHERRY_ML, Switches:CHERRY_ML, F.Cu at (71.0, 90.0)
- added U16: CHERRY_ML, Switches:CHERRY_ML, F.Cu at (66.0, 103.0)
- added U17: CHERRY_ML, Switches:CHERRY_ML, F.Cu at (102.0, 51.0)
- added U18: CHERRY_ML, Switches:CHERRY_ML, F.Cu at (97.0, 64.0)
- added U19: CHERRY_ML, Switches:CHERRY_ML, F.Cu at (92.0, 77.0)
- added U2: CHERRY_ML, Switches:CHERRY_ML, F.Cu at (53.0, 56.0)
- added U20: CHERRY_ML, Switches:CHERRY_ML, F.Cu at (87.0, 90.0)
- added U21: CHERRY_ML, Switches:CHERRY_ML, F.Cu at (82.0, 103.0)
- added U22: CHERRY_ML, Switches:CHERRY_ML, F.Cu at (115.0, 58.0)
- added U23: CHERRY_ML, Switches:CHERRY_ML, F.Cu at (110.0, 71.0)
- added U24: CHERRY_ML, Switches:CHERRY_ML, F.Cu at (105.0, 84.0)
- added U25: CHERRY_ML, Switches:CHERRY_ML, F.Cu at (100.0, 97.0)
- added U26: CHERRY_ML, Switches:CHERRY_ML, F.Cu at (95.0, 110.0)
- added U27: CHERRY_ML, Switches:CHERRY_ML, F.Cu at (129.0, 63.0)
- added U28: CHERRY_ML, Switches:CHERRY_ML, F.Cu at (124.0, 76.0)
- added U29: CHERRY_ML, Switches:CHERRY_ML, F.Cu at (119.0, 89.0)
- added U3: CHERRY_ML, Switches:CHERRY_ML, F.Cu at (48.0, 69.0)
- added U30: CHERRY_ML, Switches:CHERRY_ML, F.Cu at (114.0, 102.0)
- added U31: CHERRY_ML, Switches:CHERRY_ML, F.Cu at (109.0, 115.0)
- added U32: CHERRY_ML, Switches:CHERRY_ML, F.Cu at (160.0, 66.8)
- added U33: CHERRY_ML, Switches:CHERRY_ML, F.Cu at (162.0, 84.0)
- added U34: CHERRY_ML, Switches:CHERRY_ML, F.Cu at (169.0, 99.0)
- added U35: CHERRY_ML, Switches:CHERRY_ML, F.Cu at (178.0, 111.0)
- added U36: CHERRY_ML, Switches:CHERRY_ML, F.Cu at (184.0, 126.0)
- added U37: CHERRY_ML, Switches:CHERRY_ML, F.Cu at (182.0, 66.0)
- added U38: CHERRY_ML, Switches:CHERRY_ML, F.Cu at (185.0, 84.0)
- added U39: CHERRY_ML, Switches:CHERRY_ML, F.Cu at (191.0, 97.0)
- added U4: CHERRY_ML, Switches:CHERRY_ML, F.Cu at (43.0, 82.0)
- added U40: CHERRY_ML, Switches:CHERRY_ML, F.Cu at (199.0, 112.0)
- added U41: CHERRY_ML, Switches:CHERRY_ML, F.Cu at (201.0, 130.0)
- added U42: CHERRY_ML, Switches:CHERRY_ML, F.Cu at (206.0, 63.8)
- added U43: CHERRY_ML, Switches:CHERRY_ML, F.Cu at (206.0, 83.0)
- added U44: CHERRY_ML, Switches:CHERRY_ML, F.Cu at (212.0, 98.0)
- added U45: CHERRY_ML, Switches:CHERRY_ML, F.Cu at (220.0, 114.0)
- added U46: CHERRY_ML, Switches:CHERRY_ML, F.Cu at (221.0, 131.0)
- added U47: CHERRY_ML, Switches:CHERRY_ML, F.Cu at (224.0, 63.0)
- added U48: CHERRY_ML, Switches:CHERRY_ML, F.Cu at (226.0, 83.0)
- added U49: CHERRY_ML, Switches:CHERRY_ML, F.Cu at (230.0, 98.0)
- added U5: CHERRY_ML, Switches:CHERRY_ML, F.Cu at (38.0, 95.0)
- added U50: CHERRY_ML, Switches:CHERRY_ML, F.Cu at (240.0, 114.0)
- added U51: CHERRY_ML, Switches:CHERRY_ML, F.Cu at (240.0, 132.0)
- added U52: CHERRY_ML, Switches:CHERRY_ML, F.Cu at (243.0, 63.0)
- added U53: CHERRY_ML, Switches:CHERRY_ML, F.Cu at (243.0, 83.0)
- added U54: CHERRY_ML, Switches:CHERRY_ML, F.Cu at (247.0, 98.0)
- added U55: CHERRY_ML, Switches:CHERRY_ML, F.Cu at (256.0, 116.0)
- added U56: CHERRY_ML, Switches:CHERRY_ML, F.Cu at (257.0, 133.0)
- added U57: CHERRY_ML, Switches:CHERRY_ML, F.Cu at (266.0, 64.0)
- added U58: CHERRY_ML, Switches:CHERRY_ML, F.Cu at (261.0, 82.8)
- added U59: CHERRY_ML, Switches:CHERRY_ML, F.Cu at (266.0, 98.0)
- added U6: CHERRY_ML, Switches:CHERRY_ML, F.Cu at (33.0, 108.0)
- added U60: CHERRY_ML, Switches:CHERRY_ML, F.Cu at (276.0, 116.0)
- added U61: CHERRY_ML, Switches:CHERRY_ML, F.Cu at (278.0, 133.0)
- added U7: CHERRY_ML, Switches:CHERRY_ML, F.Cu at (69.0, 56.0)
- added U8: CHERRY_ML, Switches:CHERRY_ML, F.Cu at (64.0, 69.0)
- added U9: CHERRY_ML, Switches:CHERRY_ML, F.Cu at (59.0, 82.0)
- moved U1 25.2 mm to (139.0, 110.0)
Other:
- board size 230 x 70 mm -> 230 x 90 mm

Commit message: more keys
Parts:
- added C1: 12p, Capacitor_SMD:C_0603_1608Metric, B.Cu at (141.0, 110.0)
- added C2: 12p, Capacitor_SMD:C_0603_1608Metric, B.Cu at (137.0, 110.0)
- added C3: 100n, Capacitor_SMD:C_0603_1608Metric, B.Cu at (136.0, 143.0)
- added C4: 100n, Capacitor_SMD:C_0603_1608Metric, B.Cu at (137.0, 102.0)
- added C5: 100n, Capacitor_SMD:C_0603_1608Metric, B.Cu at (146.0, 98.0)
- added C6: 100n, Capacitor_SMD:C_0603_1608Metric, B.Cu at (143.0, 88.0)
- added C7: 100n, Capacitor_SMD:C_0603_1608Metric, B.Cu at (132.0, 91.0)
- added D61: 1N4148, Diode_SMD:D_SOD-123, B.Cu at (37.0, 131.0)
- added D62: 1N4148, Diode_SMD:D_SOD-123, B.Cu at (51.0, 131.0)
- added D63: 1N4148, Diode_SMD:D_SOD-123, B.Cu at (65.0, 131.0)
- added D64: 1N4148, Diode_SMD:D_SOD-123, B.Cu at (79.0, 131.0)
- added D65: 1N4148, Diode_SMD:D_SOD-123, B.Cu at (93.0, 131.0)
- added D66: 1N4148, Diode_SMD:D_SOD-123, B.Cu at (122.0, 127.0)
- added D67: 1N4148, Diode_SMD:D_SOD-123, B.Cu at (156.0, 127.0)
- added D68: 1N4148, Diode_SMD:D_SOD-123, B.Cu at (187.0, 131.0)
- added D69: 1N4148, Diode_SMD:D_SOD-123, B.Cu at (201.0, 131.0)
- added D70: 1N4148, Diode_SMD:D_SOD-123, B.Cu at (215.0, 131.0)
- added D71: 1N4148, Diode_SMD:D_SOD-123, B.Cu at (229.0, 131.0)
- added D72: 1N4148, Diode_SMD:D_SOD-123, B.Cu at (243.0, 131.0)
- added D73: 1N4148, Diode_SMD:D_SOD-123, B.Cu at (37.0, 145.0)
- added D74: 1N4148, Diode_SMD:D_SOD-123, B.Cu at (51.0, 145.0)
- added D75: 1N4148, Diode_SMD:D_SOD-123, B.Cu at (65.0, 145.0)
- added D76: 1N4148, Diode_SMD:D_SOD-123, B.Cu at (79.0, 145.0)
- added D77: 1N4148, Diode_SMD:D_SOD-123, B.Cu at (93.3, 145.0)
- added D78: 1N4148, Diode_SMD:D_SOD-123, B.Cu at (107.0, 145.0)
- added D79: 1N4148, Diode_SMD:D_SOD-123, B.Cu at (173.0, 145.0)
- added D80: 1N4148, Diode_SMD:D_SOD-123, B.Cu at (187.0, 145.0)
- added D81: 1N4148, Diode_SMD:D_SOD-123, B.Cu at (201.0, 145.0)
- added D82: 1N4148, Diode_SMD:D_SOD-123, B.Cu at (215.0, 145.0)
- added D83: 1N4148, Diode_SMD:D_SOD-123, B.Cu at (229.0, 145.0)
- added D84: 1N4148, Diode_SMD:D_SOD-123, B.Cu at (243.0, 145.0)
- added D85: LED_Small_ALT, LED_THT:LED_D3.0mm, F.Cu at (114.0, 44.0)
- added D86: LED_Small_ALT, LED_THT:LED_D3.0mm, F.Cu at (124.0, 44.0)
- added D87: LED_Small_ALT, LED_THT:LED_D3.0mm, F.Cu at (152.0, 44.0)
- added D88: LED_Small_ALT, LED_THT:LED_D3.0mm, F.Cu at (162.0, 44.0)
- added D89: 1N4148, Diode_SMD:D_SOD-123, B.Cu at (37.0, 52.0)
- added D90: 1N4148, Diode_SMD:D_SOD-123, B.Cu at (37.0, 66.0)
- added D91: 1N4148, Diode_SMD:D_SOD-123, B.Cu at (243.0, 52.0)
- added D92: 1N4148, Diode_SMD:D_SOD-123, B.Cu at (243.0, 66.0)
- added J1: JTAG, Connector_PinHeader_1.27mm:PinHeader_2x05_P1.27mm_Vertical, B.Cu at (154.0, 147.0)
- added J2: USB_B_Micro, Connector_USB:USB_Micro-B_Molex-105017-0001, B.Cu at (139.0, 43.7)
- added J3: Conn_01x04, Connector_PinHeader_2.54mm:PinHeader_1x04_P2.54mm_Vertical, B.Cu at (135.0, 49.0)
- added R1: 330, Resistor_SMD:R_0603_1608Metric, B.Cu at (114.0, 46.8)
- added R2: 330, Resistor_SMD:R_0603_1608Metric, B.Cu at (124.0, 46.8)
- added R3: 330, Resistor_SMD:R_0603_1608Metric, B.Cu at (152.0, 47.0)
- added R4: 330, Resistor_SMD:R_0603_1608Metric, B.Cu at (162.0, 47.0)
- added R5: 10k, Resistor_SMD:R_0603_1608Metric, B.Cu at (143.0, 143.0)
- added SW1: BOOT, Button_Switch_SMD:SW_SPST_B3U-1000P, B.Cu at (143.0, 146.0)
- added SW2: RESET, Button_Switch_SMD:SW_SPST_B3U-1000P, B.Cu at (136.0, 146.0)
- added U62: CHERRY_ML, Switches:CHERRY_ML, F.Cu at (33.0, 126.0)
- added U63: CHERRY_ML, Switches:CHERRY_ML, F.Cu at (47.0, 126.0)
- added U64: CHERRY_ML, Switches:CHERRY_ML, F.Cu at (61.0, 126.0)
- added U65: CHERRY_ML, Switches:CHERRY_ML, F.Cu at (75.0, 126.0)
- added U66: CHERRY_ML, Switches:CHERRY_ML, F.Cu at (89.0, 126.0)
- added U67: CHERRY_ML, Switches:CHERRY_ML, F.Cu at (126.0, 122.0)
- added U68: CHERRY_ML, Switches:CHERRY_ML, F.Cu at (152.0, 122.0)
- added U69: CHERRY_ML, Switches:CHERRY_ML, F.Cu at (191.0, 126.0)
- added U70: CHERRY_ML, Switches:CHERRY_ML, F.Cu at (205.0, 126.0)
- added U71: CHERRY_ML, Switches:CHERRY_ML, F.Cu at (219.0, 126.0)
- added U72: CHERRY_ML, Switches:CHERRY_ML, F.Cu at (233.0, 126.0)
- added U73: CHERRY_ML, Switches:CHERRY_ML, F.Cu at (247.0, 126.0)
- added U74: CHERRY_ML, Switches:CHERRY_ML, F.Cu at (33.0, 140.0)
- added U75: CHERRY_ML, Switches:CHERRY_ML, F.Cu at (47.0, 140.0)
- added U76: CHERRY_ML, Switches:CHERRY_ML, F.Cu at (61.0, 140.0)
- added U77: CHERRY_ML, Switches:CHERRY_ML, F.Cu at (75.0, 140.0)
- added U78: CHERRY_ML, Switches:CHERRY_ML, F.Cu at (89.0, 140.0)
- added U79: CHERRY_ML, Switches:CHERRY_ML, F.Cu at (103.0, 140.0)
- added U80: CHERRY_ML, Switches:CHERRY_ML, F.Cu at (177.0, 140.0)
- added U81: CHERRY_ML, Switches:CHERRY_ML, F.Cu at (191.0, 140.0)
- added U82: CHERRY_ML, Switches:CHERRY_ML, F.Cu at (205.0, 140.0)
- added U83: CHERRY_ML, Switches:CHERRY_ML, F.Cu at (219.0, 140.0)
- added U84: CHERRY_ML, Switches:CHERRY_ML, F.Cu at (233.0, 140.0)
- added U85: CHERRY_ML, Switches:CHERRY_ML, F.Cu at (247.0, 140.0)
- added U86: CHERRY_ML, Switches:CHERRY_ML, F.Cu at (33.0, 47.0)
- added U87: CHERRY_ML, Switches:CHERRY_ML, F.Cu at (33.0, 61.0)
- added U88: CHERRY_ML, Switches:CHERRY_ML, F.Cu at (247.0, 47.0)
- added U89: CHERRY_ML, Switches:CHERRY_ML, F.Cu at (247.0, 61.0)
- added X1: 8 MHz, Crystal:Crystal_SMD_5032-2Pin_5.0x3.2mm, B.Cu at (139.0, 107.0)
- moved U57 41.8 mm to (225.0, 56.0), turned to 20 degrees
- moved U60 41.7 mm to (240.0, 95.0), turned to 20 degrees
- moved U50 41.6 mm to (206.0, 90.0), turned to 20 degrees
- moved U61 41.4 mm to (245.0, 108.0), turned to 20 degrees
- moved U51 41.0 mm to (211.0, 103.0), turned to 20 degrees
- moved D49 40.8 mm to (203.0, 95.0)
- moved D50 40.3 mm to (208.0, 108.0)
- moved D56 39.6 mm to (223.0, 62.0)
- moved D59 39.4 mm to (238.0, 101.0)
- moved D60 39.2 mm to (243.0, 114.0)
- moved U55 38.3 mm to (224.0, 95.0), turned to 20 degrees
- moved U45 37.6 mm to (191.0, 90.0), turned to 20 degrees
- moved U46 37.5 mm to (196.0, 103.0), turned to 20 degrees
- moved U56 37.5 mm to (229.0, 108.0), turned to 20 degrees
- moved D54 36.3 mm to (221.7, 101.0)
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Connections:
- net Net-(U1-Pad10) renamed /DBG_TX
- net Net-(U1-Pad11) renamed /DBG_RX
- net Net-(U1-Pad12) renamed /TX
- net Net-(U1-Pad13) renamed /RX
- U1 pad 1: Net-(U1-Pad1) -> +3V3
- U1 pad 23: Net-(U1-Pad23) -> GND
- U1 pad 24: Net-(U1-Pad24) -> +3V3
- U1 pad 32: Net-(U1-Pad32) -> /USBD-
- U1 pad 33: Net-(U1-Pad33) -> /USBD+
- U1 pad 34: Net-(U1-Pad34) -> /SWDIO
- U1 pad 35: Net-(U1-Pad35) -> GND
- U1 pad 36: Net-(U1-Pad36) -> +3V3
- U1 pad 37: Net-(U1-Pad37) -> /SWCLK
- U1 pad 47: Net-(U1-Pad47) -> GND
- U1 pad 48: Net-(U1-Pad48) -> +3V3
- U1 pad 8: Net-(U1-Pad8) -> GND
- U1 pad 9: Net-(U1-Pad9) -> +3V3
- U2 pad 1: /ROW0 -> /ROW1
- U2 pad 3: /ROW0 -> /ROW1
- U3 pad 1: /ROW0 -> /ROW2
- U3 pad 3: /ROW0 -> /ROW2
- U4 pad 1: /ROW0 -> /ROW3
- U4 pad 3: /ROW0 -> /ROW3
- U5 pad 1: /ROW0 -> /ROW4
- U5 pad 3: /ROW0 -> /ROW4
- U6 pad 1: /ROW0 -> /ROW5
- U6 pad 3: /ROW0 -> /ROW5
Other:
- board size 230 x 90 mm -> 230 x 110 mm

Commit message: route a few columns
Parts:
- C1, C2, C3, C4, C5, C6, C7, D1, D10, D11, D12, D13, D14, D15, D16, D17, D18, D19, D2, D20, D21, D22, D23, D24, D25, D26, D27, D28, D29, D3, D30, D31, D32, D33, D34, D35, D36, D37, D38, D39, D4, D40, D41, D42, D43, D44, D45, D46, D47, D48, D49, D5, D50, D51, D52, D53, D54, D55, D56, D57, D58, D59, D6, D60, D61, D62, D63, D64, D65, D66, D67, D68, D69, D7, D70, D71, D72, D73, D74, D75, D76, D77, D78, D79, D8, D80, D81, D82, D83, D84, D89, D9, D90, D91, D92, J1, J2, J3, R1, R2, R3, R4, R5, SW1, SW2, U1, X1: moved to F.Cu
- D85, D86, D87, D88, U10, U11, U12, U13, U14, U15, U16, U17, U18, U19, U2, U20, U21, U22, U23, U24, U25, U26, U27, U28, U29, U3, U30, U31, U32, U33, U34, U35, U36, U37, U38, U39, U4, U40, U41, U42, U43, U44, U45, U46, U47, U48, U49, U5, U50, U51, U52, U53, U54, U55, U56, U57, U58, U59, U6, U60, U61, U62, U63, U64, U65, U66, U67, U68, U69, U7, U70, U71, U72, U73, U74, U75, U76, U77, U78, U79, U8, U80, U81, U82, U83, U84, U85, U86, U87, U88, U89, U9: moved to B.Cu
- moved D72 216.0 mm to (27.0, 131.0)
- moved D84 216.0 mm to (27.0, 145.0)
- moved U73 216.0 mm to (31.0, 126.0), turned to 180 degrees
- moved U85 216.0 mm to (31.0, 140.0), turned to 180 degrees
- moved U88 216.0 mm to (31.0, 47.0), turned to 180 degrees
- moved U89 216.0 mm to (31.0, 61.0), turned to 180 degrees
- moved D60 215.0 mm to (28.0, 110.5)
- moved U6 212.0 mm to (245.0, 108.0), turned to 200 degrees
- moved U61 212.0 mm to (33.0, 108.0), turned to 160 degrees
- moved U62 212.0 mm to (245.0, 126.0), turned to 180 degrees
- moved U74 212.0 mm to (245.0, 140.0), turned to 180 degrees
- moved U86 212.0 mm to (245.0, 47.0), turned to 180 degrees
- moved U87 212.0 mm to (245.0, 61.0), turned to 180 degrees
- moved D5 208.0 mm to (243.0, 113.0), turned to 0 degrees
- moved D91 208.0 mm to (35.0, 52.0), turned to 180 degrees
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Connections:
- C3 pad 1: Net-(C3-Pad1) -> /NRST
- SW2 pad 2: Net-(C3-Pad1) -> /NRST
- U1 pad 7: Net-(C3-Pad1) -> /NRST
Routing:
- net Net-(U87-Pad4): track 0.00 -> 219.9 mm, vias 0 -> 2
- net /COL10: track 0.00 -> 132.0 mm
- net /COL11: track 0.00 -> 107.1 mm
- net /COL9: track 0.00 -> 67.9 mm
- net +3V3: track 0.00 -> 48.1 mm, vias 0 -> 3
- net /USBD+: track 0.00 -> 39.4 mm
- net /USBD-: track 0.00 -> 39.4 mm
- net /NRST: track 0.00 -> 28.5 mm, vias 0 -> 2
- net Net-(U86-Pad4): track 0.00 -> 24.7 mm
- net Net-(U88-Pad4): track 0.00 -> 21.2 mm
- net GND: track 0.00 -> 20.8 mm, vias 0 -> 6
- net Net-(U49-Pad4): track 0.00 -> 18.5 mm
- net Net-(U50-Pad4): track 0.00 -> 18.4 mm
- net Net-(U51-Pad4): track 0.00 -> 18.4 mm
- net Net-(U47-Pad4): track 0.00 -> 18.0 mm
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- added copper zone on B.Cu, net GND
