File: mk3/mk3.kicad_pcb (KiCad board)
At the start: 2 copper layers, 255 x 122.5 mm, 191 parts, among them J1 JTAG, J2 USB_B_Micro, J3 Conn_01x04, SW1 BOOT, SW2 RESET, U1 STM32F070CBTx, U10 CHERRY_ML, U11 CHERRY_ML, U14 CHERRY_ML, U15 CHERRY_ML, U16 CHERRY_ML, U19 CHERRY_ML, U2 CHERRY_ML, U20 CHERRY_ML, U21 CHERRY_ML, U24 CHERRY_ML, U25 CHERRY_ML, U26 CHERRY_ML, U29 CHERRY_ML, U30 CHERRY_ML, U31 CHERRY_ML, U33 CHERRY_ML, U34 CHERRY_ML, U35 CHERRY_ML, U36 CHERRY_ML, U38 CHERRY_ML, U39 CHERRY_ML, U4 CHERRY_ML, U40 CHERRY_ML, U43 CHERRY_ML, U44 CHERRY_ML, U45 CHERRY_ML, U48 CHERRY_ML, U49 CHERRY_ML, U5 CHERRY_ML, U50 CHERRY_ML, U51 CHERRY_ML, U53 CHERRY_ML, U54 CHERRY_ML, U55 CHERRY_ML, U56 CHERRY_ML, U58 CHERRY_ML, U59 CHERRY_ML, U6 CHERRY_ML, U60 CHERRY_ML, U61 CHERRY_ML, U7 CHERRY_ML, U9 CHERRY_ML, X1 8 MHz

Commit message: add another key column to left side of layout
Parts:
- added D71: 1N4148, Diode_SMD:D_SOD-123, B.Cu at (35.5, 68.0)
- added D72: 1N4148, Diode_SMD:D_SOD-123, B.Cu at (35.5, 86.0)
- added D73: 1N4148, Diode_SMD:D_SOD-123, B.Cu at (35.5, 104.0)
- added D74: 1N4148, Diode_SMD:D_SOD-123, B.Cu at (35.5, 122.0)
- added D75: 1N4148, Diode_SMD:D_SOD-123, B.Cu at (35.5, 140.0)
- added D76: 1N4148, Diode_SMD:D_SOD-123, B.Cu at (35.5, 158.0)
- added S43: CHERRY_ML, Switches:KAILH_1350, F.Cu at (40.5, 60.0)
- added S44: CHERRY_ML, Switches:KAILH_1350, F.Cu at (40.5, 78.0)
- added S45: CHERRY_ML, Switches:KAILH_1350, F.Cu at (40.5, 96.0)
- added U12: CHERRY_ML, Switches:KAILH_1350, F.Cu at (40.5, 150.0)
- added U3: CHERRY_ML, Switches:KAILH_1350, F.Cu at (40.5, 114.0)
- added U8: CHERRY_ML, Switches:KAILH_1350, F.Cu at (40.5, 132.0)
- moved D85 148.4 mm to (97.5, 32.0)
- moved D86 148.4 mm to (107.5, 32.0)
- moved R1 148.4 mm to (97.5, 34.8)
- moved R2 148.4 mm to (107.5, 34.8)
- moved D87 135.1 mm to (120.0, 32.0)
- moved D88 135.1 mm to (130.0, 32.0)
- moved R3 135.1 mm to (120.0, 35.0)
- moved R4 135.1 mm to (130.0, 35.0)
- moved C7 99.7 mm to (68.5, 27.5), turned to 180 degrees
- moved SW2 93.9 mm to (85.5, 38.0), turned to 180 degrees
- moved C4 90.6 mm to (57.5, 32.5), turned to 270 degrees
- moved C2 89.9 mm to (51.5, 33.0), turned to 270 degrees
- moved C3 89.5 mm to (83.5, 40.5), turned to 0 degrees
- moved U1 88.9 mm to (64.5, 34.5), turned to 0 degrees
- moved X1 87.0 mm to (54.5, 35.0), turned to 90 degrees
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Routing:
- net /USBD-: track 39.4 -> 4.32 mm
- net /USBD+: track 39.4 -> 4.34 mm
- net /NRST: track 28.5 -> 18.5 mm, vias 2 -> 0
- net /SWCLK: track 12.0 -> 4.29 mm
- net /SWDIO: track 10.1 -> 5.83 mm
- net +3V3: track 48.1 -> 45.2 mm
Other:
- board size 255 x 122.5 mm -> 285 x 110.5 mm
- board text added: "BONUS"
- board text added: "DELETE"
- board text added: "END"
- board text added: "HOME"
- board text added: "INSERT"
- board text removed: "BONUS1"
- board text removed: "BONUS2"

Commit message: route a few columns of keys
Parts:
- moved C1 167.0 mm to (218.5, 40.0)
- moved C2 167.0 mm to (218.5, 36.0)
- moved C3 167.0 mm to (250.5, 43.5)
- moved C4 167.0 mm to (224.5, 35.5)
- moved C5 167.0 mm to (228.0, 44.5)
- moved C6 167.0 mm to (238.5, 41.0)
- moved C7 167.0 mm to (235.5, 30.5)
- moved J1 167.0 mm to (241.0, 42.0)
- moved J2 167.0 mm to (245.3, 30.6)
- moved J3 167.0 mm to (241.2, 36.0)
- moved R5 167.0 mm to (228.0, 46.5)
- moved SW1 167.0 mm to (224.5, 45.5)
- moved SW2 167.0 mm to (252.5, 41.0)
- moved U1 167.0 mm to (231.5, 37.5)
- moved X1 167.0 mm to (221.5, 38.0)
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Routing:
- net /ROW0: track 0.00 -> 118.9 mm
- net /ROW3: track 0.00 -> 105.5 mm
- net /ROW2: track 0.00 -> 94.1 mm
- net /ROW1: track 0.00 -> 94.1 mm
- net /COLA: track 0.00 -> 90.0 mm
- net /COL2: track 0.00 -> 90.0 mm
- net /COL1: track 0.00 -> 90.0 mm
- net /COL0: track 0.00 -> 90.0 mm
- net /ROW5: track 0.00 -> 86.6 mm
- net /ROW4: track 0.00 -> 86.1 mm
- net Net-(D72-Pad2): track 0.00 -> 3.38 mm
- net Net-(D90-Pad2): track 0.00 -> 3.18 mm
- net Net-(D8-Pad2): track 0.00 -> 3.18 mm
- net Net-(D7-Pad2): track 0.00 -> 3.18 mm
- net Net-(D61-Pad2): track 0.00 -> 3.18 mm
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
Commit message: place/route keyswitches and diodes
Parts:
- moved D43 1.92 mm to (203.5, 120.5), turned to 180 degrees
- moved D100 1.58 mm to (298.5, 156.5), turned to 180 degrees
- moved D16 1.58 mm to (108.5, 84.5), turned to 180 degrees
- moved D17 1.58 mm to (108.5, 102.5), turned to 180 degrees
- moved D18 1.58 mm to (108.5, 120.5), turned to 180 degrees
- moved D19 1.58 mm to (108.5, 138.5), turned to 180 degrees
- moved D20 1.58 mm to (108.5, 156.5), turned to 180 degrees
- moved D21 1.58 mm to (127.5, 84.5), turned to 180 degrees
- moved D22 1.58 mm to (127.5, 102.5), turned to 180 degrees
- moved D23 1.58 mm to (127.5, 120.5), turned to 180 degrees
- moved D24 1.58 mm to (127.5, 138.5), turned to 180 degrees
- moved D25 1.58 mm to (127.5, 156.5), turned to 180 degrees
- moved D26 1.58 mm to (146.5, 84.5), turned to 180 degrees
- moved D27 1.58 mm to (146.5, 102.5), turned to 180 degrees
- moved D28 1.58 mm to (146.5, 120.5), turned to 180 degrees
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Connections:
- S10 pad 3: Net-(S10-Pad3) -> /ROW1
- S10 pad 4: Net-(S10-Pad4) -> /ROW1
- S10 pad 5: Net-(S10-Pad5) -> /ROW1
- S11 pad 3: Net-(S11-Pad3) -> /ROW1
- S11 pad 4: Net-(S11-Pad4) -> /ROW1
- S11 pad 5: Net-(S11-Pad5) -> /ROW1
- S12 pad 3: Net-(S12-Pad3) -> /ROW1
- S12 pad 4: Net-(S12-Pad4) -> /ROW1
- S12 pad 5: Net-(S12-Pad5) -> /ROW1
- S13 pad 3: Net-(S13-Pad3) -> /ROW1
- S13 pad 4: Net-(S13-Pad4) -> /ROW1
- S13 pad 5: Net-(S13-Pad5) -> /ROW1
- S14 pad 3: Net-(S14-Pad3) -> /ROW1
- S14 pad 4: Net-(S14-Pad4) -> /ROW1
- S14 pad 5: Net-(S14-Pad5) -> /ROW1
- S15 pad 3: Net-(S15-Pad3) -> /ROW1
- S15 pad 4: Net-(S15-Pad4) -> /ROW1
- S15 pad 5: Net-(S15-Pad5) -> /ROW1
- S16 pad 3: Net-(S16-Pad3) -> /ROW1
- S16 pad 4: Net-(S16-Pad4) -> /ROW1
- S16 pad 5: Net-(S16-Pad5) -> /ROW1
- S21 pad 3: Net-(S21-Pad3) -> /ROW2
- S21 pad 4: Net-(S21-Pad4) -> /ROW2
- S21 pad 5: Net-(S21-Pad5) -> /ROW2
- S22 pad 3: Net-(S22-Pad3) -> /ROW2
- S22 pad 4: Net-(S22-Pad4) -> /ROW2
- S22 pad 5: Net-(S22-Pad5) -> /ROW2
- S23 pad 3: Net-(S23-Pad3) -> /ROW1
- S23 pad 4: Net-(S23-Pad4) -> /ROW1
- S23 pad 5: Net-(S23-Pad5) -> /ROW1
- S24 pad 3: Net-(S24-Pad3) -> /ROW2
- S24 pad 4: Net-(S24-Pad4) -> /ROW2
- S24 pad 5: Net-(S24-Pad5) -> /ROW2
- S25 pad 3: Net-(S25-Pad3) -> /ROW3
- S25 pad 4: Net-(S25-Pad4) -> /ROW3
- S25 pad 5: Net-(S25-Pad5) -> /ROW3
- S26 pad 3: Net-(S26-Pad3) -> /ROW4
- S26 pad 4: Net-(S26-Pad4) -> /ROW4
- S26 pad 5: Net-(S26-Pad5) -> /ROW4
- S27 pad 5: /ROW0 -> Net-(S27-Pad5)
- S28 pad 3: Net-(S28-Pad3) -> /ROW1
- S28 pad 4: Net-(S28-Pad4) -> /ROW1
- S29 pad 3: Net-(S29-Pad3) -> /ROW2
- S29 pad 4: Net-(S29-Pad4) -> /ROW2
- S30 pad 3: Net-(S30-Pad3) -> /ROW3
- S30 pad 4: Net-(S30-Pad4) -> /ROW3
- S31 pad 3: Net-(S31-Pad3) -> /ROW4
- S31 pad 4: Net-(S31-Pad4) -> /ROW4
- S32 pad 3: Net-(S32-Pad3) -> /ROW5
- S32 pad 4: Net-(S32-Pad4) -> /ROW5
- S32 pad 5: Net-(S32-Pad5) -> /ROW5
- S33 pad 3: Net-(S33-Pad3) -> /ROW5
- S33 pad 4: Net-(S33-Pad4) -> /ROW5
- S9 pad 3: Net-(S9-Pad3) -> /ROW1
- S9 pad 4: Net-(S9-Pad4) -> /ROW1
- S9 pad 5: Net-(S9-Pad5) -> /ROW1
- U2 pad 3: Net-(U2-Pad3) -> /ROW5
- U2 pad 4: Net-(U2-Pad4) -> /ROW5
- U2 pad 5: Net-(U2-Pad5) -> /ROW5
- U24 pad 3: Net-(U24-Pad3) -> /ROW3
- U24 pad 4: Net-(U24-Pad4) -> /ROW3
- U24 pad 5: Net-(U24-Pad5) -> /ROW3
- U25 pad 3: Net-(U25-Pad3) -> /ROW4
- U25 pad 4: Net-(U25-Pad4) -> /ROW4
- U25 pad 5: Net-(U25-Pad5) -> /ROW4
- U26 pad 3: Net-(U26-Pad3) -> /ROW5
- U26 pad 4: Net-(U26-Pad4) -> /ROW5
- U26 pad 5: Net-(U26-Pad5) -> /ROW5
- U29 pad 3: Net-(U29-Pad3) -> /ROW3
- U29 pad 4: Net-(U29-Pad4) -> /ROW3
- U29 pad 5: Net-(U29-Pad5) -> /ROW3
- U30 pad 3: Net-(U30-Pad3) -> /ROW4
- U30 pad 4: Net-(U30-Pad4) -> /ROW4
- U30 pad 5: Net-(U30-Pad5) -> /ROW4
- U31 pad 3: Net-(U31-Pad3) -> /ROW5
- U31 pad 4: Net-(U31-Pad4) -> /ROW5
- U31 pad 5: Net-(U31-Pad5) -> /ROW5
- U33 pad 3: Net-(U33-Pad3) -> /ROW2
- U33 pad 4: Net-(U33-Pad4) -> /ROW2
- U33 pad 5: Net-(U33-Pad5) -> /ROW2
- U34 pad 3: Net-(U34-Pad3) -> /ROW3
- U34 pad 4: Net-(U34-Pad4) -> /ROW3
- U34 pad 5: Net-(U34-Pad5) -> /ROW3
- U35 pad 3: Net-(U35-Pad3) -> /ROW4
- U35 pad 4: Net-(U35-Pad4) -> /ROW4
- U35 pad 5: Net-(U35-Pad5) -> /ROW4
- U36 pad 3: Net-(U36-Pad3) -> /ROW5
- U36 pad 4: Net-(U36-Pad4) -> /ROW5
- U36 pad 5: Net-(U36-Pad5) -> /ROW5
- U38 pad 3: Net-(U38-Pad3) -> /ROW2
- U38 pad 4: Net-(U38-Pad4) -> /ROW2
- U38 pad 5: Net-(U38-Pad5) -> /ROW2
- U39 pad 3: Net-(U39-Pad3) -> /ROW3
- U39 pad 4: Net-(U39-Pad4) -> /ROW3
- U39 pad 5: Net-(U39-Pad5) -> /ROW3
- U40 pad 3: Net-(U40-Pad3) -> /ROW4
- U40 pad 4: Net-(U40-Pad4) -> /ROW4
- U40 pad 5: Net-(U40-Pad5) -> /ROW4
- U43 pad 3: Net-(U43-Pad3) -> /ROW2
- U43 pad 4: Net-(U43-Pad4) -> /ROW2
- U43 pad 5: Net-(U43-Pad5) -> /ROW2
- U44 pad 3: Net-(U44-Pad3) -> /ROW3
- U44 pad 4: Net-(U44-Pad4) -> /ROW3
- U44 pad 5: Net-(U44-Pad5) -> /ROW3
- U45 pad 3: Net-(U45-Pad3) -> /ROW4
- U45 pad 4: Net-(U45-Pad4) -> /ROW4
- U45 pad 5: Net-(U45-Pad5) -> /ROW4
- U48 pad 3: Net-(U48-Pad3) -> /ROW2
- U48 pad 4: Net-(U48-Pad4) -> /ROW2
- U48 pad 5: Net-(U48-Pad5) -> /ROW2
- U49 pad 3: Net-(U49-Pad3) -> /ROW3
- U49 pad 4: Net-(U49-Pad4) -> /ROW3
- U49 pad 5: Net-(U49-Pad5) -> /ROW3
- U50 pad 3: Net-(U50-Pad3) -> /ROW4
- U50 pad 4: Net-(U50-Pad4) -> /ROW4
- U50 pad 5: Net-(U50-Pad5) -> /ROW4
- U51 pad 3: Net-(U51-Pad3) -> /ROW5
- U51 pad 4: Net-(U51-Pad4) -> /ROW5
- U51 pad 5: Net-(U51-Pad5) -> /ROW5
- U53 pad 3: Net-(U53-Pad3) -> /ROW2
- U53 pad 4: Net-(U53-Pad4) -> /ROW2
- U53 pad 5: Net-(U53-Pad5) -> /ROW2
- U54 pad 3: Net-(U54-Pad3) -> /ROW3
- U54 pad 4: Net-(U54-Pad4) -> /ROW3
- U54 pad 5: Net-(U54-Pad5) -> /ROW3
- U55 pad 3: Net-(U55-Pad3) -> /ROW4
- U55 pad 4: Net-(U55-Pad4) -> /ROW4
- U55 pad 5: Net-(U55-Pad5) -> /ROW4
- U56 pad 3: Net-(U56-Pad3) -> /ROW5
- U56 pad 4: Net-(U56-Pad4) -> /ROW5
- U56 pad 5: Net-(U56-Pad5) -> /ROW5
- U58 pad 3: Net-(U58-Pad3) -> /ROW2
- U58 pad 4: Net-(U58-Pad4) -> /ROW2
- U58 pad 5: Net-(U58-Pad5) -> /ROW2
- U59 pad 3: Net-(U59-Pad3) -> /ROW3
- U59 pad 4: Net-(U59-Pad4) -> /ROW3
- U59 pad 5: Net-(U59-Pad5) -> /ROW3
- U60 pad 3: Net-(U60-Pad3) -> /ROW4
- U60 pad 4: Net-(U60-Pad4) -> /ROW4
- U60 pad 5: Net-(U60-Pad5) -> /ROW4
- U61 pad 3: Net-(U61-Pad3) -> /ROW5
- U61 pad 4: Net-(U61-Pad4) -> /ROW5
- U61 pad 5: Net-(U61-Pad5) -> /ROW5
- U7 pad 3: Net-(U7-Pad3) -> /ROW5
- U7 pad 4: Net-(U7-Pad4) -> /ROW5
- U7 pad 5: Net-(U7-Pad5) -> /ROW5
Routing:
- net /ROW5: track 86.6 -> 360.5 mm
- net /ROW4: track 86.1 -> 352.0 mm
- net /ROW2: track 94.1 -> 360.0 mm
- net /ROW1: track 94.1 -> 360.0 mm
- net /ROW3: track 105.5 -> 360.0 mm
- net /ROW0: track 118.9 -> 368.5 mm
- net /COL10: track 0.00 -> 90.3 mm
- net /COL6: track 0.00 -> 90.3 mm
- net /COL9: track 0.00 -> 90.0 mm
- net /COL8: track 0.00 -> 90.0 mm
- net /COL7: track 0.00 -> 90.0 mm
- net /COL5: track 0.00 -> 90.0 mm
- net /COL4: track 0.00 -> 90.0 mm
- net /COL3: track 0.00 -> 90.0 mm
- net /COL13: track 0.00 -> 90.0 mm
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
Commit message: start routing columns
Parts:
- moved R1 109.7 mm to (255.5, 32.5), turned to 180 degrees
- moved D85 108.6 mm to (254.5, 30.0)
- moved R2 101.2 mm to (262.0, 32.5), turned to 180 degrees
- moved D86 100.1 mm to (261.0, 30.0)
- moved R3 92.7 mm to (268.5, 32.5), turned to 180 degrees
- moved D87 91.6 mm to (267.5, 30.0)
- moved R4 84.3 mm to (275.0, 32.5), turned to 180 degrees
- moved D88 83.2 mm to (274.0, 30.0)
Routing:
- net /COLA: track 90.0 -> 278.5 mm
- net /COL0: track 90.0 -> 257.1 mm
- net /COL1: track 90.0 -> 237.9 mm
- net /COL2: track 90.0 -> 220.3 mm
- net /COL3: track 90.0 -> 202.0 mm
- net /COL4: track 90.0 -> 180.6 mm
- net /COL5: track 90.0 -> 161.2 mm
- net /COL6: track 90.3 -> 142.1 mm
- net /COL7: track 90.0 -> 121.5 mm
- net Net-(R5-Pad1): track 11.6 -> 4.96 mm
Other:
- board size 285 x 110.5 mm -> 285 x 135 mm

Commit message: a bit of place/route for the MCU section
Parts:
- moved R5 34.0 mm to (260.5, 56.5), turned to 0 degrees
- moved SW1 33.2 mm to (255.5, 57.5), turned to 180 degrees
- moved C1 30.5 mm to (247.5, 49.5)
- moved C2 30.5 mm to (247.5, 45.5)
- moved C4 30.5 mm to (253.5, 45.0)
- moved C5 30.5 mm to (257.0, 54.0)
- moved C6 30.5 mm to (267.5, 50.5)
- moved C7 30.5 mm to (264.5, 40.0)
- moved J1 30.5 mm to (270.0, 51.5)
- moved J2 30.5 mm to (274.3, 40.1)
- moved J3 30.5 mm to (270.2, 45.5)
- moved U1 30.5 mm to (260.5, 47.0)
- moved X1 30.5 mm to (250.5, 47.5)
- moved SW2 28.7 mm to (279.8, 49.9), turned to 270 degrees
- moved D85 28.0 mm to (281.0, 39.0)
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Connections:
- U1 pad 45: Net-(U1-Pad45) -> /COL11
- U1 pad 46: Net-(U1-Pad46) -> /ROW0
Routing:
- net /COL11: track 90.0 -> 112.0 mm
- net /ROW0: track 368.5 -> 382.8 mm
- net /USBD+: track 4.34 -> 16.2 mm
- net /USBD-: track 4.32 -> 15.4 mm
- net /NRST: track 18.5 -> 28.5 mm, vias 0 -> 2
- net /COL10: track 90.3 -> 98.0 mm
- net /SWCLK: track 4.29 -> 10.6 mm
- net GND: track 20.6 -> 25.0 mm
- net /SWDIO: track 5.83 -> 9.93 mm
- net +3V3: track 45.2 -> 49.2 mm
- net Net-(R5-Pad1): track 4.96 -> 8.09 mm

Commit message: finish first attempt at place and route
Parts:
- removed D86, D87, D88: LED_Small_ALT, LED_THT:LED_D3.0mm
- removed R2, R3, R4: 330, Resistor_SMD:R_0603_1608Metric
- added C10: 10u, Capacitor_SMD:C_0805_2012Metric, B.Cu at (270.0, 38.0)
- added C8: 100n, Capacitor_SMD:C_0603_1608Metric, B.Cu at (273.5, 42.0)
- added C9: 100n, Capacitor_SMD:C_0603_1608Metric, B.Cu at (270.0, 40.0)
- added J4: DEBUG, Connector_PinHeader_2.54mm:PinHeader_2x03_P2.54mm_Vertical, F.Cu at (244.5, 46.5)
- added U13: TPS70933, Package_TO_SOT_SMD:SOT-23-5, B.Cu at (270.5, 43.0)
- moved R1 61.0 mm to (221.0, 42.5)
- moved D85 61.0 mm to (220.0, 39.5)
- moved J2 5.00 mm to (279.3, 40.1)
- moved J3 5.00 mm to (275.2, 45.5)
- moved D91 2.50 mm to (258.0, 66.5), turned to 0 degrees
- moved C1 1.50 mm to (247.5, 51.0)
- moved C2 1.50 mm to (247.5, 47.0)
- moved J1 1.50 mm to (270.0, 50.0)
- moved X1 1.50 mm to (250.5, 49.0)
- moved R5 1.12 mm to (260.0, 57.5)
- moved SW2 1.12 mm to (280.0, 51.0)
- moved C4 0.50 mm to (253.5, 45.5)
- moved C7 0.50 mm to (264.0, 40.0)
- moved C3 0.30 mm to (277.2, 50.5)
Connections:
- U1 pad 14: Net-(U1-Pad14) -> /COL7
- U1 pad 15: Net-(U1-Pad15) -> /COL6
- U1 pad 16: Net-(U1-Pad16) -> /COL5
- U1 pad 17: Net-(U1-Pad17) -> /COL4
- U1 pad 18: Net-(U1-Pad18) -> /COL3
- U1 pad 19: Net-(U1-Pad19) -> /COL2
- U1 pad 2: Net-(U1-Pad2) -> /COL10
- U1 pad 20: Net-(U1-Pad20) -> /COL1
- U1 pad 21: Net-(U1-Pad21) -> /COL0
- U1 pad 22: Net-(U1-Pad22) -> /COLA
- U1 pad 26: Net-(U1-Pad26) -> /LED0
- U1 pad 3: Net-(U1-Pad3) -> /COL9
- U1 pad 31: Net-(U1-Pad31) -> /COL13
- U1 pad 38: Net-(U1-Pad38) -> /COL12
- U1 pad 39: Net-(U1-Pad39) -> /ROW5
- U1 pad 4: Net-(U1-Pad4) -> /COL8
- U1 pad 40: Net-(U1-Pad40) -> /ROW4
- U1 pad 41: Net-(U1-Pad41) -> /ROW3
- U1 pad 42: Net-(U1-Pad42) -> /ROW1
- U1 pad 43: Net-(U1-Pad43) -> /ROW2
Routing:
- net /ROW5: track 360.5 -> 464.4 mm
- net /ROW4: track 352.0 -> 445.7 mm
- net /ROW3: track 360.0 -> 427.4 mm
- net /COL8: track 90.0 -> 154.9 mm
- net /COL13: track 90.0 -> 153.4 mm, vias 0 -> 2
- net /COL0: track 257.1 -> 319.7 mm
- net /COL1: track 237.9 -> 299.5 mm
- net /COLA: track 278.5 -> 339.9 mm
- net /COL2: track 220.3 -> 279.3 mm
- net /COL4: track 180.6 -> 238.9 mm
- net /COL5: track 161.2 -> 218.6 mm
- net /COL3: track 202.0 -> 259.1 mm
- net /COL7: track 121.5 -> 178.2 mm
- net /COL6: track 142.1 -> 198.7 mm
- net /LED0: track 0.00 -> 53.2 mm
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Other:
- board size 285 x 135 mm -> 285 x 125 mm

Commit message: cleanup
Parts:
- moved D76 2.83 mm to (34.5, 154.5), turned to 270 degrees
Routing:
- net /COLA: track 339.9 -> 336.5 mm
- net Net-(D76-Pad2): track 3.18 -> 4.18 mm
- net GND: vias 9 -> 18
Other:
- board size 285 x 125 mm -> 285 x 122.5 mm
- board text added: "+D-"
- board text added: "-D+"
- board text added: "3V3"
- board text added: "5V"
- board text added: "DRX"
- board text added: "DTX"
- board text added: "GND"
- board text added: "RX"
- board text added: "TX"
